File: Electronics/Mainboard/Mainboard.kicad_pcb (KiCad board)
At the start: 4 copper layers, 55 x 78 mm, 111 parts, among them U1 LM334M, U2 LMV324A, U3 LM334M, U4 LMV324A, U5 Electrosmith_Daisy_Seed_Rev4

Commit message: Rev B Mainboard and demo firmware
Parts:
- removed C3, C4: 20n, Capacitor_SMD:C_0805_2012Metric
- removed C7, C8: 10n, Capacitor_SMD:C_0805_2012Metric
- added Q1: 2N7002, Package_TO_SOT_SMD:SOT-23, F.Cu at (146.8, 106.8)
- added R35: 100k, Resistor_SMD:R_0805_2012Metric, F.Cu at (193.9, 119.9)
- added R36: 100k, Resistor_SMD:R_0805_2012Metric, F.Cu at (194.1, 92.7)
- added R37: 5M6, Resistor_SMD:R_0805_2012Metric, F.Cu at (190.4, 130.9)
- added R38: 4k7, Resistor_SMD:R_0805_2012Metric, F.Cu at (187.3, 133.7)
- added R39: 4k7, Resistor_SMD:R_0805_2012Metric, F.Cu at (145.9, 88.5)
- added R40: 4k7, Resistor_SMD:R_0805_2012Metric, F.Cu at (145.9, 101.9)
- added R41: 1M, Resistor_SMD:R_0805_2012Metric, F.Cu at (149.9, 109.6)
- added R42: 330, Resistor_SMD:R_0805_2012Metric, F.Cu at (145.9, 110.5)
- added TP22: TestPoint_Small, TestPoint:TestPoint_THTPad_D2.0mm_Drill1.0mm, F.Cu at (183.6, 106.6)
- added TP44: TestPoint_Small, TestPoint:TestPoint_THTPad_D2.0mm_Drill1.0mm, F.Cu at (183.6, 133.7)
- added TP45: TestPoint_Small, TestPoint:TestPoint_THTPad_D2.0mm_Drill1.0mm, F.Cu at (143.3, 85.9)
- added TP46: TestPoint_Small, TestPoint:TestPoint_THTPad_D2.0mm_Drill1.0mm, F.Cu at (143.3, 89.4)
- added TP47: TestPoint_Small, TestPoint:TestPoint_THTPad_D2.0mm_Drill1.0mm, F.Cu at (143.3, 93.0)
- added TP48: TestPoint_Small, TestPoint:TestPoint_THTPad_D2.0mm_Drill1.0mm, F.Cu at (143.3, 97.4)
- added TP49: TestPoint_Small, TestPoint:TestPoint_THTPad_D2.0mm_Drill1.0mm, F.Cu at (143.3, 101.0)
- added TP50: TestPoint_Small, TestPoint:TestPoint_THTPad_D2.0mm_Drill1.0mm, F.Cu at (143.3, 104.5)
- added TP51: TestPoint_Small, TestPoint:TestPoint_THTPad_D2.0mm_Drill1.0mm, F.Cu at (143.3, 109.6)
- added TP52: TestPoint_Small, TestPoint:TestPoint_THTPad_D2.0mm_Drill1.0mm, F.Cu at (143.3, 112.6)
- R1: value 1M -> 4k7
- R10, R11, R27: value 11k -> 10k
- R17: value 1M -> 10k
- R24, R4: value 612 -> 820
- R25, R9: value 6k12 -> 10k
- R26: value 11k -> 5M6
- RV1, RV2: value 100k -> 500
- TP1, TP10, TP11, TP12, TP13, TP15, TP16, TP18, TP19, TP2, TP20, TP21, TP23, TP24, TP25, TP26, TP27, TP28, TP29, TP3, TP30, TP31, TP32, TP33, TP34, TP35, TP36, TP37, TP38, TP39, TP4, TP40, TP41, TP42, TP43, TP5, TP6, TP7, TP8, TP9: footprint TestPoint:TestPoint_THTPad_D1.5mm_Drill0.7mm -> TestPoint:TestPoint_THTPad_D2.0mm_Drill1.0mm
- TP14, TP17: footprint TestPoint:TestPoint_THTPad_D1.0mm_Drill0.5mm -> TestPoint:TestPoint_THTPad_D2.0mm_Drill1.0mm
- moved RV1 42.3 mm to (191.7, 76.5), turned to 90 degrees
- moved R17 37.2 mm to (185.8, 103.8), turned to 90 degrees
- moved TP9 35.7 mm to (143.3, 116.3)
- moved R1 33.3 mm to (187.1, 106.6), turned to 180 degrees
- moved TP10 31.0 mm to (143.3, 118.9)
- moved R11 30.7 mm to (188.1, 103.8), turned to 90 degrees
- moved R27 28.2 mm to (186.1, 130.9), turned to 90 degrees
- moved R10 22.3 mm to (188.2, 130.9), turned to 90 degrees
- moved R26 20.8 mm to (190.4, 103.8), turned to 90 degrees
- moved RV2 20.3 mm to (171.9, 76.6), turned to 90 degrees
- moved TP2 20.1 mm to (148.0, 139.7)
- moved TP1 19.1 mm to (151.5, 139.7)
- moved R31 18.7 mm to (161.0, 134.7)
- moved F1 18.2 mm to (159.0, 134.7)
- moved TP13 18.0 mm to (155.1, 139.7)
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Connections:
- R1 pad 2: GND -> Net-(D6-K)
- R10 pad 1: Net-(R1-Pad1) -> Net-(R10-Pad1)
- R10 pad 2: Net-(C4-Pad1) -> Net-(U2C-+)
- R11 pad 1: Net-(C4-Pad1) -> Net-(R1-Pad1)
- R11 pad 2: Net-(U2C-+) -> Net-(U4C-+)
- R17 pad 1: Net-(R17-Pad1) -> Net-(D6-K)
- R17 pad 2: GND -> Net-(U4C--)
- R24 pad 2: Net-(D6-A) -> Net-(R24-Pad2)
- R26 pad 1: Net-(R17-Pad1) -> +5V
- R26 pad 2: Net-(C3-Pad1) -> Net-(U4C-+)
- R27 pad 1: Net-(C3-Pad1) -> Net-(D1-K)
- R27 pad 2: Net-(U4C-+) -> Net-(U2C--)
- R4 pad 2: Net-(D1-A) -> Net-(R4-Pad2)
- RV1 pad 1: Net-(C5-Pad2) -> Net-(R4-Pad2)
- RV1 pad 2: Net-(C5-Pad2) -> Net-(D1-A)
- RV1 pad 3: Net-(U2A--) -> Net-(D1-A)
- RV2 pad 1: Net-(C6-Pad2) -> Net-(R24-Pad2)
- RV2 pad 2: Net-(C6-Pad2) -> Net-(D6-A)
- RV2 pad 3: Net-(U4A--) -> Net-(D6-A)
- TP10 pad 1: Net-(U2C--) -> Net-(U5-I2C1_SDA)
- TP3 pad 1: Net-(D1-K) -> Net-(R10-Pad1)
- TP4 pad 1: Net-(R1-Pad1) -> Net-(D1-K)
- TP5 pad 1: Net-(D6-K) -> Net-(R1-Pad1)
- TP8 pad 1: Net-(R17-Pad1) -> Net-(D6-K)
- TP9 pad 1: Net-(U4C--) -> Net-(U5-I2C1_SCL)
- U2 pad 8: Net-(U2C--) -> Net-(U5-USART1_TX)
- U4 pad 8: Net-(U4C--) -> Net-(U5-USART1_RX)
- U5 pad 22: Net-(U2C--) -> Net-(D1-K)
- U5 pad 23: Net-(U4C--) -> Net-(D6-K)
- U5 pad 3: unconnected-(U5-SD_DATA_2-Pad3) -> Net-(U5-SD_DATA_2)
- U5 pad 4: unconnected-(U5-SD_DATA_1-Pad4) -> Net-(U5-SD_DATA_1)
- U5 pad 5: unconnected-(U5-SD_DATA_0-Pad5) -> Net-(Q1-G)
Routing:
- net Net-(D6-K): track 4.37 -> 111.0 mm, vias 0 -> 2
- net Net-(D1-K): track 4.74 -> 98.0 mm
- net Net-(R10-Pad1): track 0.00 -> 71.9 mm, vias 0 -> 2
- net Net-(U5-USART1_RX): track 3.18 -> 57.4 mm, vias 0 -> 3
- net Net-(U4C--): track 53.9 -> 3.89 mm
- net +3.3V: track 59.6 -> 11.4 mm, vias 3 -> 7
- net Net-(R17-Pad1): track 38.9 -> 0.00 mm, vias 1 -> 0
- net Net-(U5-USART1_TX): track 3.18 -> 41.7 mm, vias 0 -> 1
- net Net-(U2C--): track 27.8 -> 3.56 mm
- net Net-(U5-ADC_4): track 35.3 -> 16.6 mm
- net Net-(Q1-G): track 0.00 -> 15.7 mm
- net Net-(U5-SD_DATA_1): track 0.00 -> 14.4 mm
- net Net-(C4-Pad1): track 14.2 -> 0.00 mm
- net Net-(R1-Pad1): track 54.6 -> 68.8 mm, vias 1 -> 2
- net Net-(U5-I2C1_SCL): track 49.7 -> 63.7 mm
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- added copper zone on B.Cu, net +3.3V
Other:
- board size 55 x 78 mm -> 65 x 78 mm
- board text added: "3V3A"
- board text added: "AUX LED"
- board text added: "PG1"
- board text added: "PG2"
- board text added: "SG-2 Mainboard Rev B 05/2024 AJS"
- board text added: "SIG GND"
- board text added: "TOUCH 1"
- board text added: "TOUCH 2"
- board text added: "TOUCH 3"
- board text removed: "GND SIG"
- board text removed: "RX"
- board text removed: "SG-2 Mainboard Rev A 04/2024 AJS"
- board text removed: "TOUCH"
- board text removed: "TX"
