File: Electronics/Mainboard/Mainboard.kicad_sch (KiCad schematic)
At the start: 111 parts, among them U1 LM334M, U2 LMV324A, U3 LM334M, U4 LMV324A, U5 Electrosmith_Daisy_Seed_Rev4

Commit message: Rev B Mainboard and demo firmware
Parts:
- removed C3, C4: 20n, Capacitor_SMD:C_0805_2012Metric, symbol Device:C
- removed C7, C8: 10n, Capacitor_SMD:C_0805_2012Metric, symbol Device:C
- added Q1: 2N7002, Package_TO_SOT_SMD:SOT-23, symbol Transistor_FET:2N7002
- added R35, R36: 100k, Resistor_SMD:R_0805_2012Metric, symbol Device:R
- added R37: 5M6, Resistor_SMD:R_0805_2012Metric, symbol Device:R
- added R38: 4k7 0.1%, Resistor_SMD:R_0805_2012Metric, symbol Device:R
- added R39, R40: 4k7, Resistor_SMD:R_0805_2012Metric, symbol Device:R
- added R41: 1M, Resistor_SMD:R_0805_2012Metric, symbol Device:R
- added R42: 330, Resistor_SMD:R_0805_2012Metric, symbol Device:R
- added TP22, TP44, TP45, TP46, TP47, TP48, TP49, TP50, TP51, TP52: TestPoint_Small, TestPoint:TestPoint_THTPad_D2.0mm_Drill1.0mm, symbol Connector:TestPoint_Small
- R1: value 1M -> 4k7 0.1%
- R10, R11, R27: value 11k -> 10k
- R12: value 330R -> 330
- R17: value 1M -> 10k
- R24, R4: value 612 -> 820
- R25, R9: value 6k12 -> 10k
- R26: value 11k -> 5M6
- RV1, RV2: value 100k -> 500
- TP1, TP10, TP11, TP12, TP13, TP15, TP16, TP18, TP19, TP2, TP20, TP21, TP23, TP24, TP25, TP26, TP27, TP28, TP29, TP3, TP30, TP31, TP32, TP33, TP34, TP35, TP36, TP37, TP38, TP39, TP4, TP40, TP41, TP42, TP43, TP5, TP6, TP7, TP8, TP9: footprint TestPoint:TestPoint_THTPad_D1.5mm_Drill0.7mm -> TestPoint:TestPoint_THTPad_D2.0mm_Drill1.0mm
- TP14, TP17: footprint TestPoint:TestPoint_THTPad_D1.0mm_Drill0.5mm -> TestPoint:TestPoint_THTPad_D2.0mm_Drill1.0mm
- renumbered U4 to U2, U2 to U4
Connections:
- net +3.3V: now also R39.1, R40.1, R42.1
- net +5V: now also R26.1, R37.1, TP45.1, TP48.1
- net GND: now also Q1.2 (S), R41.2, TP47.1, TP50.1; no longer R1.2, R17.2
- net at D6.1 (K), R25.2: now also R1.2, R17.1, TP8.1, U5.23 (ADC_1), TP22.1; no longer TP5.1
- net at D6.2 (A), U3.2, U3.3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: now also RV2.2, RV2.3; no longer R24.2
- net at R29.2, TP33.1, U5.13 (I2C1_SDA): now also TP10.1
- net at R28.2, TP32.1, U5.12 (I2C1_SCL): now also TP9.1
- net at D1.1 (K), R9.2: now also R27.1, TP4.1, U5.22 (ADC_0), R38.2, TP44.1; no longer TP3.1
- net at R10.2: now also U2.10 (+), R37.2; no longer R11.1
- net at R11.2, U4.10 (+): now also R26.2
- net at D1.2 (A), U1.2, U1.3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: now also RV1.2, RV1.3; no longer R4.2
- net at C5.2, TP14.1, U2.1: now also R35.1; no longer RV1.1, RV1.2
- net at R2.2, U2.2 (-): now also R35.2; no longer RV1.3
- net at C6.2, TP17.1, U4.1: now also R36.1; no longer RV2.1, RV2.2
- net at R3.2, U4.2 (-): now also R36.2; no longer RV2.3
- net at R27.2: now also U2.9 (-); no longer U2.10 (+)
- net at TP31.1, U5.15 (USART1_RX): now also U4.8
- net at TP30.1, U5.14 (USART1_TX): now also U2.8
- net at U5.3 (SD_DATA_2): now also R39.2, TP46.1
- net at U5.4 (SD_DATA_1): now also R40.2, TP49.1
- net at U5.5 (SD_DATA_0): now also Q1.1 (G), R41.1
- new net: R24.2, RV2.1
- new net: R10.1, R38.1, TP3.1
- new net: R4.2, RV1.1
- new net: Q1.3 (D), TP52.1
- new net: R42.2, TP51.1
- new net: R1.1, R11.1, TP5.1
- new net: R17.2, U4.9 (-)
Other:
- note added: "Adjust RV1 for 3.3V at TP44"
- note added: "Adjust RV2 for 3.3V at TP22"
- note added: "Aux. LED"
- note added: "Daisy Seed"
- note added: "I2C"
- note added: "Pitch gate 1"
- note added: "Pitch gate 2"
- note added: "SG-2 Mainboard Rev B"
- note added: "Touch input 1"
- note added: "Touch input 2"
- note added: "Touch input 3"
- note removed: "220uA current source"
- note removed: "Aux serial out"
- note removed: "Daisy Seed and decoupling"
- note removed: "SG-2 Mainboard Rev A"
- note removed: "Touch input"
- moved on the sheet: C17, C18, D1, D6, R24, R25, R34, R4, R9, RV1, RV2, TP1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
